Commit message: code: sync from learning-os-from-arduino@c9e5ece

File: code/13_quadruped/arduino_os_quad_robot/urdf/arduino_os_quad_robot.urdf (robot description, URDF)
Before this commit: robot arduino_os_quad_robot, 17 links, 16 joints
Links:
- removed link FL_foot
- removed link FL_hip_servo
- removed link FL_knee_servo
- removed link FL_thigh
- removed link FR_foot
- removed link FR_hip_servo
- removed link FR_knee_servo
- removed link FR_thigh
- removed link RL_foot
- removed link RL_hip_servo
- removed link RL_knee_servo
- removed link RL_thigh
- removed link RR_foot
- removed link RR_hip_servo
- removed link RR_knee_servo
- removed link RR_thigh
- added link Assem130_5__STS3215_03a_nopassivehorn_1, mass 0.055; collision mesh filename=package://arduino_os_quad_robot/meshes/Assem130__STS3215_03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; visual mesh filename=package://arduino_os_quad_robot/meshes/Assem130__STS3215_03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
- added link Assem130_5__STS3215_03a_nopassivehorn_3, mass 0.055; collision mesh filename=package://arduino_os_quad_robot/meshes/Assem130__STS3215_03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; visual mesh filename=package://arduino_os_quad_robot/meshes/Assem130__STS3215_03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
- added link Assem130_5__bracket_outline_1, mass 0.0194513; collision mesh filename=package://arduino_os_quad_robot/meshes/Assem130__bracket_ou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; visual mesh filename=package://arduino_os_quad_robot/meshes/Assem130__bracket_ou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
- added link Assem130_5__leg_link1_2, mass 0.0402227; collision mesh filename=package://arduino_os_quad_robot/meshes/Assem130__leg_link1_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; visual mesh filename=package://arduino_os_quad_robot/meshes/Assem130__leg_link1_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
- added link Assem130_6__STS3215_03a_nopassivehorn_1, mass 0.055; collision mesh filename=package://arduino_os_quad_robot/meshes/Assem130__STS3215_03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; visual mesh filename=package://arduino_os_quad_robot/meshes/Assem130__STS3215_03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
- added link Assem130_6__STS3215_03a_nopassivehorn_3, mass 0.055; collision mesh filename=package://arduino_os_quad_robot/meshes/Assem130__STS3215_03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; visual mesh filename=package://arduino_os_quad_robot/meshes/Assem130__STS3215_03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
- added link Assem130_6__bracket_outline_1, mass 0.0194513; collision mesh filename=package://arduino_os_quad_robot/meshes/Assem130__bracket_ou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; visual mesh filename=package://arduino_os_quad_robot/meshes/Assem130__bracket_ou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
- added link Assem130_6__leg_link1_2, mass 0.0402227; collision mesh filename=package://arduino_os_quad_robot/meshes/Assem130__leg_link1_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; visual mesh filename=package://arduino_os_quad_robot/meshes/Assem130__leg_link1_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
- added link Assem130_right_5__STS3215_03a_nopassivehorn_1, mass 0.055; collision mesh filename=package://arduino_os_quad_robot/meshes/Assem130__STS3215_03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; visual mesh filename=package://arduino_os_quad_robot/meshes/Assem130__STS3215_03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
- added link Assem130_right_5__STS3215_03a_nopassivehorn_3, mass 0.055; collision mesh filename=package://arduino_os_quad_robot/meshes/Assem130__STS3215_03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; visual mesh filename=package://arduino_os_quad_robot/meshes/Assem130__STS3215_03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
- added link Assem130_right_5__bracket_outline_1, mass 0.0194513; collision mesh filename=package://arduino_os_quad_robot/meshes/Assem130__bracket_ou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; visual mesh filename=package://arduino_os_quad_robot/meshes/Assem130__bracket_ou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
- added link Assem130_right_5__leg_link1_2, mass 0.0402227; collision mesh filename=package://arduino_os_quad_robot/meshes/Assem130__leg_link1_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; visual mesh filename=package://arduino_os_quad_robot/meshes/Assem130__leg_link1_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
- added link Assem130_right_6__STS3215_03a_nopassivehorn_1, mass 0.055; collision mesh filename=package://arduino_os_quad_robot/meshes/Assem130__STS3215_03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; visual mesh filename=package://arduino_os_quad_robot/meshes/Assem130__STS3215_03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
- added link Assem130_right_6__STS3215_03a_nopassivehorn_3, mass 0.055; collision mesh filename=package://arduino_os_quad_robot/meshes/Assem130__STS3215_03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; visual mesh filename=package://arduino_os_quad_robot/meshes/Assem130__STS3215_03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
- added link Assem130_right_6__bracket_outline_1, mass 0.0194513; collision mesh filename=package://arduino_os_quad_robot/meshes/Assem130__bracket_ou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; visual mesh filename=package://arduino_os_quad_robot/meshes/Assem130__bracket_ou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
- added link Assem130_right_6__leg_link1_2, mass 0.0402227; collision mesh filename=package://arduino_os_quad_robot/meshes/Assem130__leg_link1_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; visual mesh filename=package://arduino_os_quad_robot/meshes/Assem130__leg_link1_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
Joints:
- removed joint FL_hip_joint
- removed joint FL_hip_mount
- removed joint FL_knee_joint
- removed joint FL_knee_mount
- removed joint FR_hip_joint
- removed joint FR_hip_mount
- removed joint FR_knee_joint
- removed joint FR_knee_mount
- removed joint RL_hip_joint
- removed joint RL_hip_mount
- removed joint RL_knee_joint
- removed joint RL_knee_mount
- removed joint RR_hip_joint
- removed joint RR_hip_mount
- removed joint RR_knee_joint
- removed joint RR_knee_mount
- added joint Assem130_5__STS3215_03a_nopassivehorn_1__Assem130_5__leg_link1_2: type revolute, parent Assem130_5__STS3215_03a_nopassivehorn_1, child Assem130_5__leg_link1_2, origin xyz=0.01188538639 -2.538415101e-08 0.01742230355 rpy=-1.570796327 0 -0.9503346526, axis 0 1 0, limit lower=-2 upper=2 effort=2.942 velocity=4.717
- added joint Assem130_5__STS3215_03a_nopassivehorn_3__Assem130_5__bracket_outline_1: type revolute, parent Assem130_5__STS3215_03a_nopassivehorn_3, child Assem130_5__bracket_outline_1, origin xyz=0.01188538639 -2.538415101e-08 0.01742230355 rpy=-1.570796327 0 -2.521130979, axis 0 1 0, limit lower=-2 upper=2 effort=2.942 velocity=4.717
- added joint Assem130_5__leg_link1_2__Assem130_5__STS3215_03a_nopassivehorn_3: type fixed, parent Assem130_5__leg_link1_2, child Assem130_5__STS3215_03a_nopassivehorn_3, origin xyz=-0.06223680659 -0.03027769645 0.04447477731 rpy=-1.570796327 -0.6204616742 -3.141592653, axis 0 0 1
- added joint Assem130_6__STS3215_03a_nopassivehorn_1__Assem130_6__leg_link1_2: type revolute, parent Assem130_6__STS3215_03a_nopassivehorn_1, child Assem130_6__leg_link1_2, origin xyz=0.01188538639 -2.538415101e-08 0.01742230355 rpy=-1.570796327 0 -0.9503346526, axis 0 1 0, limit lower=-2 upper=2 effort=2.942 velocity=4.717
- added joint Assem130_6__STS3215_03a_nopassivehorn_3__Assem130_6__bracket_outline_1: type revolute, parent Assem130_6__STS3215_03a_nopassivehorn_3, child Assem130_6__bracket_outline_1, origin xyz=0.01188538639 -2.538415101e-08 0.01742230355 rpy=-1.570796327 0 -2.521130979, axis 0 1 0, limit lower=-2 upper=2 effort=2.942 velocity=4.717
- added joint Assem130_6__leg_link1_2__Assem130_6__STS3215_03a_nopassivehorn_3: type fixed, parent Assem130_6__leg_link1_2, child Assem130_6__STS3215_03a_nopassivehorn_3, origin xyz=-0.06223680659 -0.03027769645 0.04447477731 rpy=-1.570796327 -0.6204616742 -3.141592653, axis 0 0 1
- added joint Assem130_right_5__STS3215_03a_nopassivehorn_1__Assem130_right_5__leg_link1_2: type revolute, parent Assem130_right_5__STS3215_03a_nopassivehorn_1, child Assem130_right_5__leg_link1_2, origin xyz=0.01188538639 -2.538415101e-08 0.01742230355 rpy=1.570796327 0 0.9503346526, axis 0 -1 0, limit lower=-2 upper=2 effort=2.942 velocity=4.717
- added joint Assem130_right_5__STS3215_03a_nopassivehorn_3__Assem130_right_5__bracket_outline_1: type revolute, parent Assem130_right_5__STS3215_03a_nopassivehorn_3, child Assem130_right_5__bracket_outline_1, origin xyz=0.01188538639 -2.538415101e-08 0.01742230355 rpy=1.570796327 0 2.521130979, axis 0 -1 0, limit lower=-2 upper=2 effort=2.942 velocity=4.717
- added joint Assem130_right_5__leg_link1_2__Assem130_right_5__STS3215_03a_nopassivehorn_3: type fixed, parent Assem130_right_5__leg_link1_2, child Assem130_right_5__STS3215_03a_nopassivehorn_3, origin xyz=-0.06223677708 0.03027769645 0.04447481861 rpy=1.570796327 -0.6204616742 3.141592653, axis 0 0 1
- added joint Assem130_right_6__STS3215_03a_nopassivehorn_1__Assem130_right_6__leg_link1_2: type revolute, parent Assem130_right_6__STS3215_03a_nopassivehorn_1, child Assem130_right_6__leg_link1_2, origin xyz=0.01188538639 -2.538415101e-08 0.01742230355 rpy=1.570796327 0 0.9503346526, axis 0 -1 0, limit lower=-2 upper=2 effort=2.942 velocity=4.717
- added joint Assem130_right_6__STS3215_03a_nopassivehorn_3__Assem130_right_6__bracket_outline_1: type revolute, parent Assem130_right_6__STS3215_03a_nopassivehorn_3, child Assem130_right_6__bracket_outline_1, origin xyz=0.01188538639 -2.538415101e-08 0.01742230355 rpy=1.570796327 0 2.521130979, axis 0 -1 0, limit lower=-2 upper=2 effort=2.942 velocity=4.717
- added joint Assem130_right_6__leg_link1_2__Assem130_right_6__STS3215_03a_nopassivehorn_3: type fixed, parent Assem130_right_6__leg_link1_2, child Assem130_right_6__STS3215_03a_nopassivehorn_3, origin xyz=-0.06223677708 0.03027769645 0.04447481861 rpy=1.570796327 -0.6204616742 3.141592653, axis 0 0 1
- added joint body_1__Assem130_5__STS3215_03a_nopassivehorn_1: type fixed, parent base_link, child Assem130_5__STS3215_03a_nopassivehorn_1, origin xyz=0.07811461361 0.03537769645 0.01642997462 rpy=-1.570796327 0 0, axis 0 0 -1
- added joint body_1__Assem130_6__STS3215_03a_nopassivehorn_1: type fixed, parent base_link, child Assem130_6__STS3215_03a_nopassivehorn_1, origin xyz=-0.07188538639 0.03537769645 0.01642997462 rpy=-1.570796327 0 0, axis 0 0 -1
- added joint body_1__Assem130_right_5__STS3215_03a_nopassivehorn_1: type fixed, parent base_link, child Assem130_right_5__STS3215_03a_nopassivehorn_1, origin xyz=-0.07188538639 -0.03537769645 0.01643002538 rpy=1.570796327 0 0, axis 0 0 1
- added joint body_1__Assem130_right_6__STS3215_03a_nopassivehorn_1: type fixed, parent base_link, child Assem130_right_6__STS3215_03a_nopassivehorn_1, origin xyz=0.07811461361 -0.03537769645 0.01643002538 rpy=1.570796327 0 0, axis 0 0 1
