Commit message: code: sync from manuscript@4b6c8b8

File: code/13_quadruped/arduino_os_quad_robot/urdf/arduino_os_quad_robot_rl.urdf (robot description, URDF)
Before this commit: robot arduino_os_quad_robot, 17 links, 16 joints
Links:
- added link imu_link
- added link sensor_board; visual mesh filename=package://arduino_os_quad_robot/meshes/sensor_board.glb
Joints:
- added joint imu_joint: type fixed, parent sensor_board, child imu_link, origin xyz=0 -4.65257908e-05 -0.000545500014 rpy=3.141592654 0 0
- added joint sensor_board_mount: type fixed, parent base_link, child sensor_board, origin xyz=0.106 0 0.009 rpy=-2.35619449 0 -1.570796327
